File: tf530/eagle/SL530.sch (EAGLE design)
At the start: 42 parts, among them IC4 74LVC1G17DBV, IC5 74LVC1G17DBV, U1 LM1117, X1 MC68000

Commit message: Bit of a clean up of the silkscreen
Parts:
- removed AUXPINS: AUXPINS, SparkFun-Retired:JUMPER-2PTH
- added C14, C15: 10uF, microbuilder:CAP_CERAMIC1206
- added C16, C17: 0.1uF, SparkFun-Capacitors:0.1UF-25V(+80/-20%)(0603)
- added RCLKLOAD: INF, SparkFun-Resistors:0.05OHM-1/5W-1%(0603)
- IC3: value LM1117 -> LM1117-3.3
- R3: value 10K -> 47K
- TP1: value A500 -> TP1
- renumbered A500 to TP1, IDE to IDECONNECTOR, JP7 to PWR1, U$1 to IC8, U$2 to IC6, U$3 to IC7, U$4 to IC9, U1 to IC3
Connections:
- removed net AUX0: AUXPINS.1, XC9572XL(BUS).PB02/3
- removed net AUX1: AUXPINS.2, XC9572XL(BUS).PB04/17
- new net SPARE: XC9572XL(RAM).PB03/15
- net A14: no longer XC9572XL(BUS).PB03/12
- net A7: no longer XC9572XL(RAM).PB03/15
- net AVEC: now also XC9572XL(BUS).PB02/8; no longer XC9572XL(BUS).PB03/14
- net CLKCPU: now also RCLKLOAD.1
- net DSACK0: no longer XC9572XL(BUS).PB02/8
- net FC0: now also XC9572XL(BUS).PB03/12; no longer XC9572XL(BUS).PB03/6
- net FC1: now also XC9572XL(BUS).PB03/14; no longer XC9572XL(BUS).PB03/11
- net GND: now also C14.P$2, C15.P$2, C16.2, C17.2, RCLKLOAD.2
- net IPL1: now also XC9572XL(BUS).PB04/17
- net IPL2: now also XC9572XL(BUS).PB02/3
- net VCC: now also C14.P$1, C15.P$1, C16.1, C17.1
Other:
- note added: "C14-C17 are for tuning/stability purposes. These should not be required for normal operation but can be used to help with instability."
- note added: "OVR and INT2 are redudant. They are retained for test purposes only."
- note added: "Terrible Fire TF530 Revision 3 Copyright (C) 2017 Stephen J. Leary All Rights Reserved."
- note added: "This is now a test point. No longer required for standard operation."
- note added: "This resistor is to let me experiment with clock line loads to tune to higher clock frequencies. It is not required for 24Mhz operation"
- note added: "Without these resistor networks the control bus floats low and does not work."
